File: pcb/Adafruit PowerBoost 500 Basic Replica.sch (KiCad schematic (older format))
At the start: 32 parts, among them CN1 USBA, J1 HEADER, J2 PWR OUT, J3 Batería, Q1 MMUN2133LT1G, U1 TPS61090RSAR

Commit message: Applies Diego Corrections
Parts:
- removed FID2: U1 FID, Fiducial:Fiducial_0.5mm_Mask1mm, symbol Mechanical:Fiducial
Other:
- note added: "Fiduciales"
- note removed: "Fiducials"
Changed lines of the file:
@@
 Wire Notes Line
 	4200 1550 3350 1550
-$Comp
-L Mechanical:Fiducial FID2
-U 1 1 616E0E3E
-P 5350 2200
-F 0 "FID2" H 5435 2246 50  0000 L CNN
-F 1 "U1 FID" H 5435 2155 50  0000 L CNN
-F 2 "Fiducial:Fiducial_0.5mm_Mask1mm" H 5350 2200 50  0001 C CNN
-F 3 "~" H 5350 2200 50  0001 C CNN
-	1    5350 2200
-	1    0    0    -1
-$EndComp
-Wire Notes Line
-	4800 2450 4800 1550
 Wire Notes Line
 	4800 1550 6100 1550
 Wire Notes Line
-	6100 1550 6100 2450
-Wire Notes Line
-	6100 2450 4800 2450
+	6100 2200 4800 2200
 Text Notes 4900 1700 0    50   ~ 0
-Fiducials
+Fiduciales
 $Comp
 L Device:Q_PNP_BEC_BRT Q1
@@
 Wire Notes Line
 	8400 4000 11000 4000
+Wire Notes Line
+	6100 2200 6100 1550
+Wire Notes Line
+	4800 1550 4800 2200
 $EndSCHEMATC

Commit message: Cambios de acuerdo a checks del excel
Parts:
- CN1: Mouser N (none) -> 640-USB1130-15-A
- J2: footprint Connector_JST:JST_EH_S2B-EH_1x02_P2.50mm_Horizontal -> dci_lorsi:JST_EH_S2B-EH_1x02_P2.50mm_Horizontal
- L1: Mouser N (none) -> 810-VLC5045T-6R8M
- U1: Mouser N (none) -> 595-TPS61090RSAR; Mouser Num 595-TPS61090RSAR -> (none)
Changed lines of the file:
@@
 F 2 "Inductor_SMD:L_Taiyo-Yuden_NR-40xx_HandSoldering" H 3400 4300 50  0001 C CNN
 F 3 "~" H 3400 4300 50  0001 C CNN
+F 4 "810-VLC5045T-6R8M" H 3400 4300 50  0001 C CNN "Mouser N"
 	1    3400 4300
 	0    -1   -1   0
@@
 F 2 "Package_DFN_QFN:QFN-16-1EP_4x4mm_P0.65mm_EP2.1x2.1mm" H 4200 4500 50  0001 C CNN
 F 3 "" H 4200 4500 50  0001 C CNN
-F 4 "595-TPS61090RSAR" H 4500 4150 50  0001 C CNN "Mouser Num"
+F 4 "" H 4500 4150 50  0001 C CNN "Mouser Num"
+F 5 "595-TPS61090RSAR" H 4500 4150 50  0001 C CNN "Mouser N"
 	1    4500 4150
 	1    0    0    -1
@@
 F 0 "J2" H 7400 4300 50  0000 L CNN
 F 1 "PWR OUT" H 7300 4400 50  0000 L CNN
-F 2 "Connector_JST:JST_EH_S2B-EH_1x02_P2.50mm_Horizontal" H 7450 4200 50  0001 C CNN
+F 2 "dci_lorsi:JST_EH_S2B-EH_1x02_P2.50mm_Horizontal" H 7450 4200 50  0001 C CNN
 F 3 "~" H 7450 4200 50  0001 C CNN
 	1    7450 4200
@@
 F 2 "Connector_USB:USB_A_Molex_67643_Horizontal" H 9950 4600 50  0001 C CNN
 F 3 "" H 9950 4600 50  0001 C CNN
+F 4 "640-USB1130-15-A" H 10200 4650 50  0001 C CNN "Mouser N"
 	1    10200 4650
 	1    0    0    -1
